Commit message: 控制实际机器人

File: g01_moveit_config/config/G01.ros2_control.xacro (robot description, xacro)
@@ -1,10 +1,14 @@
 <?xml version="1.0"?>
 <robot xmlns:xacro="http://www.ros.org/wiki/xacro">
-    <xacro:macro name="G01_ros2_control" params="name initial_positions_file">
+    <xacro:macro name="G01_ros2_control" params="name initial_positions_file hardware_plugin state_topic command_topic">
         <xacro:property name="initial_positions" value="${load_yaml(initial_positions_file)['initial_positions']}"/>
         <ros2_control name="${name}" type="system">
             <hardware>
-                <!-- By default, set up controllers for simulation. This won't work on real hardware -->
-                <plugin>mock_components/GenericSystem</plugin>
+                <!-- Default: simulation / mock. For real robot, pass a different plugin via xacro args. -->
+                <plugin>${hardware_plugin}</plugin>
+                <xacro:if value="${hardware_plugin == 'g01_topic_hardware/G01TopicSystem'}">
+                    <param name="state_topic">${state_topic}</param>
+                    <param name="command_topic">${command_topic}</param>
+                </xacro:if>
             </hardware>
             <joint name="base_joint1">

File: g01_moveit_config/config/G01.urdf.xacro (robot description, xacro)
@@ -2,8 +2,16 @@
 <robot xmlns:xacro="http://www.ros.org/wiki/xacro" name="G01">
     <xacro:arg name="initial_positions_file" default="initial_positions.yaml" />
+    <xacro:arg name="ros2_control_hardware_plugin" default="mock_components/GenericSystem" />
+    <xacro:arg name="ros2_control_state_topic" default="" />
+    <xacro:arg name="ros2_control_command_topic" default="" />
     <!-- Import G01 urdf file -->
     <xacro:include filename="$(find moveit_resources_g01_description)/urdf/G01-URDF888.urdf" />
     <!-- Import control_xacro -->
     <xacro:include filename="G01.ros2_control.xacro" />
-    <xacro:G01_ros2_control name="FakeSystem" initial_positions_file="$(arg initial_positions_file)"/>
+    <xacro:G01_ros2_control
+        name="G01System"
+        initial_positions_file="$(arg initial_positions_file)"
+        hardware_plugin="$(arg ros2_control_hardware_plugin)"
+        state_topic="$(arg ros2_control_state_topic)"
+        command_topic="$(arg ros2_control_command_topic)"/>
 </robot>
