Commit message: 替换左臂1077

File: g01_moveit_config/config/G01.ros2_control.xacro (robot description, xacro)
@@ -15,4 +15,13 @@
                 </xacro:if>
             </hardware>
+            <!-- Real head feedback comes directly from comm.py. Supply a state
+                 in mock mode so FK/visualization also has a known head angle. -->
+            <xacro:if value="${hardware_plugin == 'mock_components/GenericSystem'}">
+                <joint name="head_joint">
+                    <state_interface name="position">
+                        <param name="initial_value">${initial_positions['head_joint']}</param>
+                    </state_interface>
+                </joint>
+            </xacro:if>
             <joint name="base_joint1">
                 <command_interface name="position"/>

File: moveit_resources/g01_description/urdf/G01-URDF888.urdf (robot description, URDF)
Before this commit: robot G01, 8 links, 7 joints
Joints:
- joint head_joint: axis (none) -> 0 0 -1; limit (none) -> lower=0 upper=1.0472 effort=100 velocity=100; type fixed -> revolute
