Commit message: 6.11

File: DOBOT_6Axis_ROS2/dobot_rviz/urdf/cr7_robot.urdf (robot description, URDF)
Before this commit: robot cr7_robot, 8 links, 7 joints
Joints:
- joint joint2: origin xyz=0 0 0 rpy=-1.57080420997483 1.57079631189374 -3.14158502419526 -> xyz=-0.000018278000876307487 0 0 rpy=-1.57080420997483 1.569684 -3.14158502419526
- joint joint3: origin xyz=-0.377 0 0.025 rpy=0 0 0 -> xyz=-0.37767788696289062 0 0.025569253 rpy=0 -0.00712 -0.0
- joint joint4: origin xyz=-0.306999999999969 0 0.116 rpy=0 0 -1.57079677671549 -> xyz=-0.30705142211914062 0 0.11602764129638672 rpy=0 0.006778 -1.57079677671549
- joint joint5: origin xyz=0 -0.116 0 rpy=1.5707963267949 0 0 -> xyz=-0.000033348001539707184 -0.11602764129638672 0 rpy=1.570579138 0 0
- joint joint6: origin xyz=0 0.104999656773681 0 rpy=-1.5707963267949 0 0 -> xyz=0.00019047899544239044 0.105 0 rpy=-1.5702245 0 0

Commit message: 生成变化矩阵

File: DOBOT_6Axis_ROS2/dobot_rviz/urdf/cr7_robot.urdf (robot description, URDF)
Before this commit: robot cr7_robot, 8 links, 7 joints
Joints:
- joint joint2: origin xyz=-0.000018278000876307487 0 0 rpy=-1.57080420997483 1.569684 -3.14158502419526 -> xyz=0 0 0 rpy=-1.57080420997483 1.57079631189374 -3.14158502419526
- joint joint3: origin xyz=-0.37767788696289062 0 0.025569253 rpy=0 -0.00712 -0.0 -> xyz=-0.377 0 0.025 rpy=0 0 0
- joint joint4: origin xyz=-0.30705142211914062 0 0.11602764129638672 rpy=0 0.006778 -1.57079677671549 -> xyz=-0.306999999999969 0 0.116 rpy=0 0 -1.57079677671549
- joint joint5: origin xyz=-0.000033348001539707184 -0.11602764129638672 0 rpy=1.570579138 0 0 -> xyz=0 -0.116 0 rpy=1.5707963267949 0 0
- joint joint6: origin xyz=0.00019047899544239044 0.105 0 rpy=-1.5702245 0 0 -> xyz=0 0.104999656773681 0 rpy=-1.5707963267949 0 0
