Commit message: MoveIt 错误码

File: moveit_resources/g01_description/urdf/G01-URDF888.urdf (robot description, URDF)
Before this commit: robot G01, 18 links, 17 joints
Joints:
- joint body_joint1: limit lower=-0.25 upper=0 effort=100 velocity=1 -> lower=-0.25 upper=0.0 effort=100 velocity=1

Commit message: 验证EE_LINK

File: moveit_resources/g01_description/urdf/G01-URDF888.urdf (robot description, URDF)
Before this commit: robot G01, 18 links, 17 joints
Links:
- added link l_tool
- added link r_tool
Joints:
- added joint l_tool_to_L6: type fixed, parent L6, child l_tool, origin xyz=0 0 0.15 rpy=0 0 0
- added joint r_tool_to_R6: type fixed, parent R6, child r_tool, origin xyz=0 0 0.15 rpy=0 0 0

Commit message: 实际部署

File: moveit_resources/g01_description/urdf/G01-URDF888.urdf (robot description, URDF)
Before this commit: robot G01, 20 links, 19 joints
Joints:
- joint base_joint1: limit lower=-50.0 upper=50.0 effort=100.0 velocity=1.0 -> lower=-1.0 upper=1.0 effort=100.0 velocity=1.0
- joint body_joint1: limit lower=-0.25 upper=0.0 effort=100 velocity=1 -> lower=-0.25 upper=0 effort=100 velocity=1
- joint body_joint2: limit lower=0 upper=1.5708 effort=100 velocity=2 -> lower=0 upper=1.5708 effort=100 velocity=0.26
- joint l_arm_joint1: axis 0 0 -1 -> 0 0 1; origin xyz=0 0.377999999999968 0.1205 rpy=0 0 0 -> xyz=0 0.377999999999968 0.1205 rpy=0 0 -1.57079631189374
- joint l_arm_joint2: axis 0 0 -1 -> 0 0 1; limit lower=-3.1416 upper=0.2 effort=100 velocity=2 -> lower=-3.1416 upper=3.1416 effort=100 velocity=2; origin xyz=-0.0639751221249114 0.00178430633972448 0.08299999999993 rpy=3.11370925402287 -1.57079631189374 3.14159265358979 -> xyz=-0.0639751221249114 0.00178430633972448 0.08299999999993 rpy=-1.57079631189374 0 1.57079631189374
- joint l_arm_joint3: axis 0 0 1 -> 0 0 -1; limit lower=-3.1416 upper=3.1416 effort=100 velocity=2 -> lower=-2.79 upper=2.79 effort=100 velocity=2
- joint l_arm_joint4: axis 0 0 -1 -> 0 0 1
- joint l_arm_joint5: axis 0 0 -1 -> 0 0 1
- joint l_arm_joint6: axis 0 0 -1 -> 0 0 1
- joint r_arm_joint1: origin xyz=0 0.377999999999968 -0.3085 rpy=3.14159265358979 0 3.14159265358979 -> xyz=0 0.377999999999968 -0.3085 rpy=3.14159265358979 0 1.57079631189374
- joint r_arm_joint2: limit lower=-3.1416 upper=0.2 effort=100 velocity=2 -> lower=-3.1416 upper=3.1416 effort=100 velocity=2; origin xyz=0.0639942896829944 0.000854919860884817 0.0829999999999999 rpy=0.962598114856819 1.57079631189374 0.975956634984278 -> xyz=0.0639942896829944 0.000854919860884817 0.0829999999999999 rpy=-1.57079631189374 0 -1.57079631189374
- joint r_arm_joint3: limit lower=-3.1416 upper=3.1416 effort=100 velocity=2 -> lower=-2.79 upper=2.79 effort=100 velocity=2

Commit message: 加桌子

File: moveit_resources/g01_description/urdf/G01-URDF888.urdf (robot description, URDF)
Before this commit: robot G01, 20 links, 19 joints
Links:
- link base_link: geometry collision box size=0.19 0.42 0.19; collision box size=0.34 0.35 0.51

Commit message: 修改腰部碰撞

File: moveit_resources/g01_description/urdf/G01-URDF888.urdf (robot description, URDF)
Before this commit: robot G01, 20 links, 19 joints
Links:
- link YB: geometry collision mesh filename=package://moveit_resources_g01_description/meshes/YB.STL; visual mesh filename=package://moveit_resources_g01_description/meshes/YB.STL
- link base_link: geometry collision box size=0.19 0.42 0.19; collision box size=0.34 0.35 0.51

Commit message: 增加臂基坐标系

File: moveit_resources/g01_description/urdf/G01-URDF888.urdf (robot description, URDF)
Before this commit: robot G01, 20 links, 19 joints
Links:
- added link l_base_link
- added link r_base_link
Joints:
- added joint l_base_link_to_YB: type fixed, parent YB, child l_base_link, origin xyz=0.000 0.378 0.0565 rpy=0 0 -3.1415926
- added joint r_base_link_to_YB: type fixed, parent YB, child r_base_link, origin xyz=-0.000 0.378 -0.2445 rpy=-3.1415926 0 0

Commit message: 实际控左臂

File: moveit_resources/g01_description/urdf/G01-URDF888.urdf (robot description, URDF)
Before this commit: robot G01, 22 links, 21 joints
Joints:
- joint body_joint2: limit lower=0 upper=1.5708 effort=100 velocity=0.26 -> lower=0 upper=1.5708 effort=100 velocity=0.1

Commit message: 6.5

File: moveit_resources/g01_description/urdf/G01-URDF888.urdf (robot description, URDF)
Before this commit: robot G01, 20 links, 19 joints
Links:
- added link l_base_link
- added link r_base_link
- link YB: geometry collision mesh filename=package://moveit_resources_g01_description/meshes/YB.STL; visual mesh filename=package://moveit_resources_g01_description/meshes/YB.STL
- link base_link: geometry collision box size=0.19 0.42 0.19; collision box size=0.34 0.35 0.51
Joints:
- added joint l_base_link_to_YB: type fixed, parent YB, child l_base_link, origin xyz=0.000 0.378 0.0565 rpy=0 0 -3.1415926
- added joint r_base_link_to_YB: type fixed, parent YB, child r_base_link, origin xyz=-0.000 0.378 -0.2445 rpy=-3.1415926 0 0
- joint base_joint1: limit lower=-50.0 upper=50.0 effort=100.0 velocity=1.0 -> lower=-1.0 upper=1.0 effort=100.0 velocity=1.0
- joint body_joint2: limit lower=0 upper=1.5708 effort=100 velocity=2 -> lower=0 upper=1.5708 effort=100 velocity=0.1
- joint l_arm_joint1: axis 0 0 -1 -> 0 0 1; origin xyz=0 0.377999999999968 0.1205 rpy=0 0 0 -> xyz=0 0.377999999999968 0.1205 rpy=0 0 -1.57079631189374
- joint l_arm_joint2: axis 0 0 -1 -> 0 0 1; limit lower=-3.1416 upper=0.2 effort=100 velocity=2 -> lower=-3.1416 upper=3.1416 effort=100 velocity=2; origin xyz=-0.0639751221249114 0.00178430633972448 0.08299999999993 rpy=3.11370925402287 -1.57079631189374 3.14159265358979 -> xyz=-0.0639751221249114 0.00178430633972448 0.08299999999993 rpy=-1.57079631189374 0 1.57079631189374
- joint l_arm_joint3: axis 0 0 1 -> 0 0 -1; limit lower=-3.1416 upper=3.1416 effort=100 velocity=2 -> lower=-2.79 upper=2.79 effort=100 velocity=2
- joint l_arm_joint4: axis 0 0 -1 -> 0 0 1
- joint l_arm_joint5: axis 0 0 -1 -> 0 0 1
- joint l_arm_joint6: axis 0 0 -1 -> 0 0 1
- joint r_arm_joint1: origin xyz=0 0.377999999999968 -0.3085 rpy=3.14159265358979 0 3.14159265358979 -> xyz=0 0.377999999999968 -0.3085 rpy=3.14159265358979 0 1.57079631189374
- joint r_arm_joint2: limit lower=-3.1416 upper=0.2 effort=100 velocity=2 -> lower=-3.1416 upper=3.1416 effort=100 velocity=2; origin xyz=0.0639942896829944 0.000854919860884817 0.0829999999999999 rpy=0.962598114856819 1.57079631189374 0.975956634984278 -> xyz=0.0639942896829944 0.000854919860884817 0.0829999999999999 rpy=-1.57079631189374 0 -1.57079631189374
- joint r_arm_joint3: limit lower=-3.1416 upper=3.1416 effort=100 velocity=2 -> lower=-2.79 upper=2.79 effort=100 velocity=2

Commit message: urdf碰撞模型替换

File: moveit_resources/g01_description/urdf/G01-URDF888.urdf (robot description, URDF)
Before this commit: robot G01, 22 links, 21 joints
Links:
- link L1: geometry collision cylinder length=0.170 radius=0.065; visual mesh filename=package://moveit_resources_g01_description/meshes/L1.STL
- link L2: geometry collision cylinder length=0.160 radius=0.065; collision cylinder length=0.160 radius=0.065
- link L3: geometry collision cylinder length=0.10 radius=0.065; collision cylinder length=0.140 radius=0.045
- link L4: geometry collision cylinder length=0.140 radius=0.045; visual mesh filename=package://moveit_resources_g01_description/meshes/L4.STL
- link L5: geometry collision cylinder length=0.150 radius=0.045; visual mesh filename=package://moveit_resources_g01_description/meshes/L5.STL
- link L6: geometry collision cylinder length=0.07 radius=0.045; collision cylinder length=0.10 radius=0.085
- link R1: geometry collision cylinder length=0.170 radius=0.065; visual mesh filename=package://moveit_resources_g01_description/meshes/R1.STL
- link R2: geometry collision cylinder length=0.160 radius=0.065; collision cylinder length=0.160 radius=0.065
- link R3: geometry collision cylinder length=0.10 radius=0.065; collision cylinder length=0.140 radius=0.045
- link R4: geometry collision cylinder length=0.140 radius=0.045; visual mesh filename=package://moveit_resources_g01_description/meshes/R4.STL
- link R5: geometry collision cylinder length=0.150 radius=0.045; visual mesh filename=package://moveit_resources_g01_description/meshes/R5.STL
- link R6: geometry collision cylinder length=0.07 radius=0.045; collision cylinder length=0.10 radius=0.085
- link YB: geometry collision box size=0.05 0.05 0.09; collision box size=0.23 0.51 0.32
- link base_link: geometry collision box size=0.19 0.42 0.19; collision box size=0.34 0.35 0.51
Joints:
- joint body_joint1: limit lower=-0.25 upper=0.0 effort=100 velocity=1 -> lower=-0.25 upper=0 effort=100 velocity=1
- joint body_joint2: limit lower=0 upper=1.5708 effort=100 velocity=0.1 -> lower=0 upper=1.5708 effort=100 velocity=0.26
- joint l_arm_joint1: axis 0 0 1 -> 0 0 -1
- joint l_arm_joint2: axis 0 0 1 -> 0 0 -1
- joint l_arm_joint3: axis 0 0 -1 -> 0 0 1
- joint l_arm_joint4: axis 0 0 1 -> 0 0 -1
- joint l_arm_joint5: axis 0 0 1 -> 0 0 -1
- joint l_arm_joint6: axis 0 0 1 -> 0 0 -1
- joint l_base_link_to_YB: origin xyz=0.000 0.378 0.0565 rpy=0 0 -3.1415926 -> xyz=0.000 0.378 0.056 rpy=0 0 -3.1415926
- joint r_base_link_to_YB: origin xyz=-0.000 0.378 -0.2445 rpy=-3.1415926 0 0 -> xyz=-0.000 0.378 -0.244 rpy=-3.1415926 0 0

Commit message: 修改urdf

File: moveit_resources/g01_description/urdf/G01-URDF888.urdf (robot description, URDF)
Before this commit: robot G01, 22 links, 21 joints
Joints:
- joint l_tool_to_L6: origin xyz=0 0 0.15 rpy=0 0 0 -> xyz=0 0 0.129 rpy=0 0 0
- joint r_tool_to_R6: origin xyz=0 0 0.15 rpy=0 0 0 -> xyz=0 0 0.129 rpy=0 0 0

Commit message: 碰撞模型替换

File: moveit_resources/g01_description/urdf/G01-URDF888.urdf (robot description, URDF)
Before this commit: robot G01, 22 links, 21 joints
Links:
- link L1: geometry collision cylinder length=0.170 radius=0.065; visual mesh filename=package://moveit_resources_g01_description/meshes/L1.STL
- link L2: geometry collision cylinder length=0.160 radius=0.065; collision cylinder length=0.160 radius=0.065
- link L3: geometry collision cylinder length=0.10 radius=0.065; collision cylinder length=0.140 radius=0.045
- link L4: geometry collision cylinder length=0.140 radius=0.045; visual mesh filename=package://moveit_resources_g01_description/meshes/L4.STL
- link L5: geometry collision cylinder length=0.150 radius=0.045; visual mesh filename=package://moveit_resources_g01_description/meshes/L5.STL
- link L6: geometry collision cylinder length=0.07 radius=0.045; collision cylinder length=0.10 radius=0.085
- link R1: geometry collision cylinder length=0.170 radius=0.065; visual mesh filename=package://moveit_resources_g01_description/meshes/R1.STL
- link R2: geometry collision cylinder length=0.160 radius=0.065; collision cylinder length=0.160 radius=0.065
- link R3: geometry collision cylinder length=0.10 radius=0.065; collision cylinder length=0.140 radius=0.045
- link R4: geometry collision cylinder length=0.140 radius=0.045; visual mesh filename=package://moveit_resources_g01_description/meshes/R4.STL
- link R5: geometry collision cylinder length=0.150 radius=0.045; visual mesh filename=package://moveit_resources_g01_description/meshes/R5.STL
- link R6: geometry collision cylinder length=0.07 radius=0.045; collision cylinder length=0.10 radius=0.085
- link YB: geometry collision box size=0.05 0.05 0.09; collision box size=0.23 0.51 0.32
Joints:
- joint body_joint2: limit lower=0 upper=1.5708 effort=100 velocity=0.1 -> lower=0 upper=1.5708 effort=100 velocity=0.26
- joint l_arm_joint1: axis 0 0 1 -> 0 0 -1
- joint l_arm_joint2: axis 0 0 1 -> 0 0 -1
- joint l_arm_joint3: axis 0 0 -1 -> 0 0 1
- joint l_arm_joint4: axis 0 0 1 -> 0 0 -1
- joint l_arm_joint5: axis 0 0 1 -> 0 0 -1
- joint l_arm_joint6: axis 0 0 1 -> 0 0 -1
- joint l_base_link_to_YB: origin xyz=0.000 0.378 0.0565 rpy=0 0 -3.1415926 -> xyz=0.000 0.378 0.056 rpy=0 0 -3.1415926
- joint l_tool_to_L6: origin xyz=0 0 0.129 rpy=0 0 0 -> xyz=0 0 0.15 rpy=0 0 0
- joint r_base_link_to_YB: origin xyz=-0.000 0.378 -0.2445 rpy=-3.1415926 0 0 -> xyz=-0.000 0.378 -0.244 rpy=-3.1415926 0 0
- joint r_tool_to_R6: origin xyz=0 0 0.129 rpy=0 0 0 -> xyz=0 0 0.15 rpy=0 0 0

Commit message: 放大1.05倍

File: moveit_resources/g01_description/urdf/G01-URDF888.urdf (robot description, URDF)
Before this commit: robot G01, 22 links, 21 joints
Links:
- link L1: geometry collision cylinder length=${arm_collision_scale * 0.170} radius=${arm_collision_scale * 0.065}; visual mesh filename=package://moveit_resources_g01_description/meshes/L1.STL
- link L2: geometry collision cylinder length=${arm_collision_scale * 0.160} radius=${arm_collision_scale * 0.065}; collision cylinder length=${arm_collision_scale * 0.160} radius=${arm_collision_scale * 0.065}
- link L3: geometry collision cylinder length=${arm_collision_scale * 0.10} radius=${arm_collision_scale * 0.065}; collision cylinder length=${arm_collision_scale * 0.140} radius=${arm_collision_scale * 0.045}
- link L4: geometry collision cylinder length=${arm_collision_scale * 0.140} radius=${arm_collision_scale * 0.045}; visual mesh filename=package://moveit_resources_g01_description/meshes/L4.STL
- link L5: geometry collision cylinder length=${arm_collision_scale * 0.150} radius=${arm_collision_scale * 0.045}; visual mesh filename=package://moveit_resources_g01_description/meshes/L5.STL
- link L6: geometry collision cylinder length=${arm_collision_scale * 0.07} radius=${arm_collision_scale * 0.045}; collision cylinder length=${arm_collision_scale * 0.10} radius=${arm_collision_scale * 0.085}
- link R1: geometry collision cylinder length=${arm_collision_scale * 0.170} radius=${arm_collision_scale * 0.065}; visual mesh filename=package://moveit_resources_g01_description/meshes/R1.STL
- link R2: geometry collision cylinder length=${arm_collision_scale * 0.160} radius=${arm_collision_scale * 0.065}; collision cylinder length=${arm_collision_scale * 0.160} radius=${arm_collision_scale * 0.065}
- link R3: geometry collision cylinder length=${arm_collision_scale * 0.10} radius=${arm_collision_scale * 0.065}; collision cylinder length=${arm_collision_scale * 0.140} radius=${arm_collision_scale * 0.045}
- link R4: geometry collision cylinder length=${arm_collision_scale * 0.140} radius=${arm_collision_scale * 0.045}; visual mesh filename=package://moveit_resources_g01_description/meshes/R4.STL
- link R5: geometry collision cylinder length=${arm_collision_scale * 0.150} radius=${arm_collision_scale * 0.045}; visual mesh filename=package://moveit_resources_g01_description/meshes/R5.STL
- link R6: geometry collision cylinder length=${arm_collision_scale * 0.07} radius=${arm_collision_scale * 0.045}; collision cylinder length=${arm_collision_scale * 0.10} radius=${arm_collision_scale * 0.085}

Commit message: 隔离板

File: moveit_resources/g01_description/urdf/G01-URDF888.urdf (robot description, URDF)
Before this commit: robot G01, 22 links, 21 joints
Joints:
- joint l_arm_joint1: axis 0 0 -1 -> 0 0 1
- joint l_arm_joint2: axis 0 0 -1 -> 0 0 1
- joint l_arm_joint3: axis 0 0 1 -> 0 0 -1
- joint l_arm_joint4: axis 0 0 -1 -> 0 0 1
- joint l_arm_joint5: axis 0 0 -1 -> 0 0 1
- joint l_arm_joint6: axis 0 0 -1 -> 0 0 1

Commit message: 修改末端坐标系位置

File: moveit_resources/g01_description/urdf/G01-URDF888.urdf (robot description, URDF)
Before this commit: robot G01, 22 links, 21 joints
Joints:
- joint l_tool_to_L6: origin xyz=0 0 0.15 rpy=0 0 0 -> xyz=0 0 0.13 rpy=0 0 0
- joint r_tool_to_R6: origin xyz=0 0 0.15 rpy=0 0 0 -> xyz=0 0 0.13 rpy=0 0 0

Commit message: 加入相机碰撞

File: moveit_resources/g01_description/urdf/G01-URDF888.urdf (robot description, URDF)
Before this commit: robot G01, 22 links, 21 joints
Links:
- link R6: geometry collision box size=0.12 0.05 0.015; collision cylinder length=${arm_collision_scale * 0.07} radius=${arm_collision_scale * 0.045}

Commit message: 修改urdf

File: moveit_resources/g01_description/urdf/G01-URDF888.urdf (robot description, URDF)
Before this commit: robot G01, 22 links, 21 joints
Joints:
- joint l_base_link_to_YB: origin xyz=0.000 0.378 0.056 rpy=0 0 -3.1415926 -> xyz=0.000 0.378 0.0565 rpy=0 0 -3.1415926
- joint r_base_link_to_YB: origin xyz=-0.000 0.378 -0.244 rpy=-3.1415926 0 0 -> xyz=-0.000 0.378 -0.2445 rpy=-3.1415926 0 0

Commit message: 增加struct.json文件

File: moveit_resources/g01_description/urdf/G01-URDF888.urdf (robot description, URDF)
Before this commit: robot G01, 22 links, 21 joints
Joints:
- joint l_tool_to_L6: origin xyz=0 0 0.13 rpy=0 0 0 -> xyz=0 0 0.0342 rpy=0 0 0
- joint r_tool_to_R6: origin xyz=0 0 0.13 rpy=0 0 0 -> xyz=0 0 0.0342 rpy=0 0 0

Commit message: 修改urdf

File: moveit_resources/g01_description/urdf/G01-URDF888.urdf (robot description, URDF)
Before this commit: robot G01, 22 links, 21 joints
Links:
- removed link L1
- removed link L2
- removed link L3
- removed link L4
- removed link L5
- removed link L6
- removed link R1
- removed link R2
- removed link R3
- removed link R4
- removed link R5
- removed link R6
- removed link l_base_link
- removed link l_tool
- removed link r_base_link
- removed link r_tool
Joints:
- removed joint l_arm_joint1
- removed joint l_arm_joint2
- removed joint l_arm_joint3
- removed joint l_arm_joint4
- removed joint l_arm_joint5
- removed joint l_arm_joint6
- removed joint l_base_link_to_YB
- removed joint l_tool_to_L6
- removed joint r_arm_joint1
- removed joint r_arm_joint2
- removed joint r_arm_joint3
- removed joint r_arm_joint4
- removed joint r_arm_joint5
- removed joint r_arm_joint6
- removed joint r_base_link_to_YB
- removed joint r_tool_to_R6

File: moveit_resources/g01_description/urdf/cr7_robot.urdf (robot description, URDF)
Before this commit: robot cr7_robot, 8 links, 7 joints
Links:
- removed link Link1
- removed link Link2
- removed link Link3
- removed link Link4
- removed link Link5
- removed link Link6
- removed link base_link
- removed link dummy_link
Joints:
- removed joint dummy_joint
- removed joint joint1
- removed joint joint2
- removed joint joint3
- removed joint joint4
- removed joint joint5
- removed joint joint6

Commit message: 修改腰部限制

File: moveit_resources/g01_description/urdf/G01-URDF888.urdf (robot description, URDF)
Before this commit: robot G01, 6 links, 5 joints
Joints:
- joint body_joint2: limit lower=0 upper=1.5708 effort=100 velocity=0.26 -> lower=0 upper=0.87 effort=100 velocity=0.26

Commit message: 实际测试失败率高

File: moveit_resources/g01_description/urdf/G01-URDF888.urdf (robot description, URDF)
Before this commit: robot G01, 6 links, 5 joints
Joints:
- joint body_joint2: limit lower=0 upper=0.87 effort=100 velocity=0.26 -> lower=0 upper=0.785 effort=100 velocity=0.26
