Commit message: 腰部正常运动

File: moveit_resources/g01_description/urdf/G01-URDF888.urdf (robot description, URDF)
Before this commit: robot G01, 6 links, 5 joints
Joints:
- joint body_joint1: axis 0 -1 0 -> 0 1 0; limit lower=-0.25 upper=0 effort=100 velocity=1 -> lower=0.0 upper=0.25 effort=100 velocity=1

Commit message: 修改ip

File: moveit_resources/g01_description/urdf/G01-URDF888.urdf (robot description, URDF)
Before this commit: robot G01, 6 links, 5 joints
Links:
- link YB: geometry collision box size=0.22 0.15 0.13; collision box size=0.23 0.51 0.32

Commit message: 修改可达性验证

File: moveit_resources/g01_description/urdf/G01-URDF888.urdf (robot description, URDF)
Before this commit: robot G01, 6 links, 5 joints
Joints:
- joint body_joint1: limit lower=0.0 upper=0.25 effort=100 velocity=1 -> lower=0.0 upper=0.24 effort=100 velocity=1

Commit message: 增加注释

File: moveit_resources/g01_description/urdf/G01-URDF888.urdf (robot description, URDF)
Before this commit: robot G01, 6 links, 5 joints
Links:
- link YB: geometry collision box size=0.23 0.51 0.32; visual mesh filename=package://moveit_resources_g01_description/meshes/YB.STL

Commit message: 替换新模型

File: moveit_resources/g01_description/urdf/G01-URDF888.urdf (robot description, URDF)
Before this commit: robot G01, 6 links, 5 joints
Links:
- added link base_sj, mass 19.7724725085068; collision mesh filename=package://moveit_resources_g01_description/meshes/1.STL; visual mesh filename=package://moveit_resources_g01_description/meshes/1.STL
- link SJ: mass 15.5120061335875 -> 17.1115281100298; geometry collision mesh filename=package://moveit_resources_g01_description/meshes/2.STL; visual mesh filename=package://moveit_resources_g01_description/meshes/2.STL
- link YB: mass 5.03869108075918 -> 5.10087522591895; geometry collision mesh filename=package://moveit_resources_g01_description/meshes/3.STL; visual mesh filename=package://moveit_resources_g01_description/meshes/3.STL
- link base_link: mass 24.9214864900972 -> 34.9231249877199; geometry collision mesh filename=package://moveit_resources_g01_description/meshes/base_link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; visual mesh filename=package://moveit_resources_g01_description/meshes/base_link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
Joints:
- added joint base_sj_joint: type fixed, parent base_link, child base_sj, origin xyz=0.127 0 0.1355 rpy=0 0 0, axis 0 0 0
- joint base_joint1: axis -1 0 0 -> 1 0 0
- joint base_joint2: axis 0 1 0 -> 0 0 1
- joint body_joint1: axis 0 1 0 -> 0 0 1; limit lower=0.0 upper=0.24 effort=100 velocity=1 -> lower=0 upper=0.24 effort=100 velocity=0; origin xyz=0 0.04548 0 rpy=0 0 0 -> xyz=0 0 0.043 rpy=0 0 0; parent base_link -> base_sj
- joint body_joint2: limit lower=0 upper=0.785 effort=100 velocity=0.26 -> lower=0 upper=1.4 effort=100 velocity=100; origin xyz=0 0.117000000000034 0.0940000000000007 rpy=0 0 0 -> xyz=0 0.1175 0.654 rpy=1.5708 0 -3.1416
- joint world_to_base_footprint: origin xyz=0 0 0.6 rpy=1.5708 0 3.1415926 -> xyz=0 0 0.0 rpy=0.0 0.0 0.0

Commit message: 修改交换位置

File: moveit_resources/g01_description/urdf/G01-URDF888.urdf (robot description, URDF)
Before this commit: robot G01, 7 links, 6 joints
Joints:
- joint base_sj_joint: axis 0 0 0 -> (none)

Commit message: 修改升降电机urdf抬高5mm

File: moveit_resources/g01_description/urdf/G01-URDF888.urdf (robot description, URDF)
Before this commit: robot G01, 7 links, 6 joints
Joints:
- joint body_joint1: limit lower=0 upper=0.24 effort=100 velocity=0 -> lower=0 upper=0.19 effort=100 velocity=0; origin xyz=0 0 0.043 rpy=0 0 0 -> xyz=0 0 0.048 rpy=0 0 0

Commit message: 加入物料放置碰撞

File: moveit_resources/g01_description/urdf/G01-URDF888.urdf (robot description, URDF)
Before this commit: robot G01, 7 links, 6 joints
Links:
- link base_link: geometry collision box size=0.34 0.34 0.03; collision mesh filename=package://moveit_resources_g01_description/meshes/base_link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

Commit message: 7.24

File: moveit_resources/g01_description/urdf/G01-URDF888.urdf (robot description, URDF)
Before this commit: robot G01, 7 links, 6 joints
Joints:
- joint body_joint2: limit lower=0 upper=1.4 effort=100 velocity=100 -> lower=0 upper=1 effort=100 velocity=100

Commit message: 替换碰撞模型

File: moveit_resources/g01_description/urdf/G01-URDF888.urdf (robot description, URDF)
Before this commit: robot G01, 7 links, 6 joints
Links:
- link base_link: geometry collision box size=0.34 0.34 0.035; collision mesh filename=package://moveit_resources_g01_description/meshes/base_link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

Commit message: 替换模型

File: moveit_resources/g01_description/urdf/G01-URDF888.urdf (robot description, URDF)
Before this commit: robot G01, 7 links, 6 joints
Links:
- added link head, mass 0.83283062923428; collision mesh filename=package://moveit_resources_g01_description/meshes/6.STL; visual mesh filename=package://moveit_resources_g01_description/meshes/6.STL
- link SJ: mass 17.1115281100298 -> 17.6002532483208
- link YB: mass 5.10087522591895 -> 6.37285826562377
- link base_link: mass 34.9231249877199 -> 41.5277464083994; geometry collision mesh filename=package://moveit_resources_g01_description/meshes/base_link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; visual mesh filename=package://moveit_resources_g01_description/meshes/base_link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
- link base_sj: mass 19.7724725085068 -> 19.9697634207302
Joints:
- added joint head_joint: type revolute, parent YB, child head, origin xyz=-0.047 0.5115 -0.1664 rpy=3.1416 0 3.1416, axis 0 0 1, limit lower=-1.045 upper=0 effort=100 velocity=100
- joint base_sj_joint: axis (none) -> 0 0 0; origin xyz=0.127 0 0.1355 rpy=0 0 0 -> xyz=0 0 0 rpy=0 0 0
- joint body_joint1: limit lower=0 upper=0.19 effort=100 velocity=0 -> lower=0 upper=0.19 effort=0 velocity=0; origin xyz=0 0 0.048 rpy=0 0 0 -> xyz=0.127 0 0.1355 rpy=0 0 0
- joint body_joint2: limit lower=0 upper=1 effort=100 velocity=100 -> lower=0 upper=1.0 effort=100 velocity=100; origin xyz=0 0.1175 0.654 rpy=1.5708 0 -3.1416 -> xyz=0 0.1175 0.697 rpy=1.5708 0 -3.1416

Commit message: 头部碰撞模型

File: moveit_resources/g01_description/urdf/G01-URDF888.urdf (robot description, URDF)
Before this commit: robot G01, 8 links, 7 joints
Links:
- link base_link: geometry collision box size=0.34 0.34 0.03; collision mesh filename=package://moveit_resources_g01_description/meshes/base_link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
- link head: geometry collision box size=0.26 0.2 0.2; collision mesh filename=package://moveit_resources_g01_description/meshes/6.STL
Joints:
- joint head_joint: axis 0 0 1 -> (none); limit lower=-1.045 upper=0 effort=100 velocity=100 -> (none); type revolute -> fixed

Commit message: 修复tf冲突

File: moveit_resources/g01_description/urdf/G01-URDF888.urdf (robot description, URDF)
Before this commit: robot G01, 8 links, 7 joints
Links:
- removed link base_link
- added link moveit_base_link, mass 41.5277464083994; collision box size=0.34 0.34 0.03; collision mesh filename=package://moveit_resources_g01_description/meshes/base_link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
Joints:
- joint base_joint2: child base_link -> moveit_base_link
- joint base_sj_joint: parent base_link -> moveit_base_link
